Commit message: Created a first configuration of the robot arm

File: project_workspace/src/robot_package/urdf/robot_arm.xacro (robot description, xacro)
@@ -5,4 +5,6 @@
     <xacro:include filename="$(find robot_package)/urdf/robot_parameters.xacro" />
     <!-- END - Include -->
+    <link name="world"/>
+    <!--
     <xacro:m_link_box name="${l00}"
                 origin_rpy="0 0 0" origin_xyz="0 0 0"
@@ -11,27 +13,28 @@
                 iyy="170.667" iyz="0"
                 izz="170.667"
-                size = "1 1 1"/>
+                size = "1 1 0"/>
+    -->
     <xacro:m_joint name="${l00}__${l01}"
                    type="revolute"
                    axis_xyz="0 0 1"
-                   origin_rpy="0 0 0" origin_xyz="0 0 0.5"
-                   parent="${l00}"
+                   origin_rpy="0 0 0" origin_xyz="0 0 -0.5"
+                   parent="world"
                    child="${l01}"
                    limit_e="1000"
-                   limit_l="-3.14"
-                   limit_u="3.14"
+                   limit_l="-6,28319"
+                   limit_u="6,28319"
                    limit_v="0.5"/>
     <xacro:m_link_cylinder name="${l01}"
-                origin_rpy="0 0 0" origin_xyz="0 0 0.2"
+                origin_rpy="0 0 0" origin_xyz="0 0 1"
                 mass = "157.633"
                 ixx="13.235" ixy="0" ixz="0"
                 iyy="13.235" iyz="0"
                 izz="9.655"
-                radius = "0.35"
-                length="0.4"/>
+                radius = "0.1"
+                length="2"/>
     <xacro:m_joint name="${l01}__${l02}"
                    type="revolute"
                    axis_xyz="0 1 0"
-                   origin_rpy="0 0 0" origin_xyz="0 0 0.4"
+                   origin_rpy="0 1.57 0" origin_xyz="0 0 2"
                    parent="${l01}"
                    child="${l02}"
@@ -41,11 +44,29 @@
                    limit_v="0.5"/>
     <xacro:m_link_cylinder name="${l02}"
-                origin_rpy="0 0 0" origin_xyz="0 0 0.4"
-                mass = "57.906"
-                ixx="12.679" ixy="0" ixz="0"
-                iyy="12.679" iyz="0"
-                izz="0.651"
-                radius = "0.15"
-                length="0.8"/>
+                origin_rpy="0 0 0" origin_xyz="0 0 0.5"
+                mass = "0.1"
+                ixx="0" ixy="0" ixz="0"
+                iyy="0" iyz="0"
+                izz="0"
+                radius = "0.1"
+                length="1"/>
+    <xacro:m_joint name="${l02}__${l03}"
+                   type="revolute"
+                   axis_xyz="0 1 0"
+                   origin_rpy="0 0 0" origin_xyz="0 0 1"
+                   parent="${l02}"
+                   child="${l03}"
+                   limit_e="1000"
+                   limit_l="-3.14"
+                   limit_u="3.14"
+                   limit_v="0.5"/>
+    <xacro:m_link_cylinder name="${l03}"
+                origin_rpy="0 0 0" origin_xyz="0 0 0.5"
+                mass = "0.05"
+                ixx="0" ixy="0" ixz="0"
+                iyy="0" iyz="0"
+                izz="0"
+                radius = "0.1"
+                length="1"/>
     <gazebo>
         <plugin name ="gazebo_ros_control" filename="libgazebo_ros_control.so">

File: project_workspace/src/robot_package/urdf/robot_parameters.xacro (robot description, xacro)
@@ -4,3 +4,4 @@
   <xacro:property name="l01" value="link_01" />
   <xacro:property name="l02" value="link_02" />
+  <xacro:property name="l03" value="link_03" />
 </robot>
