Commit message: Addend end effector link

File: project_workspace/src/robot_package/urdf/links_joints.xacro (robot description, xacro)
@@ -22,4 +22,5 @@
     <xacro:macro name="m_link_cylinder" params="name origin_xyz origin_rpy radius length mass ixx ixy ixz iyy iyz izz">
         <link name="${name}">
+            <gravity>0</gravity>
             <inertial>
                 <mass value="${mass}" />

File: project_workspace/src/robot_package/urdf/robot_arm.xacro (robot description, xacro)
@@ -18,5 +18,5 @@
                    type="revolute"
                    axis_xyz="0 0 1"
-                   origin_rpy="0 0 0" origin_xyz="0 0 -0.5"
+                   origin_rpy="0 0 0" origin_xyz="0 0 0"
                    parent="world"
                    child="${l01}"
@@ -39,5 +39,5 @@
                    parent="${l01}"
                    child="${l02}"
-                   limit_e="1000"
+                   limit_e="10"
                    limit_l="-3.14"
                    limit_u="3.14"
@@ -57,5 +57,5 @@
                    parent="${l02}"
                    child="${l03}"
-                   limit_e="1000"
+                   limit_e="10"
                    limit_l="-3.14"
                    limit_u="3.14"
@@ -69,4 +69,22 @@
                 radius = "0.1"
                 length="1"/>
+     <xacro:m_joint name="${l03}__${lee}"
+                   type="revolute"
+                   axis_xyz="0 1 0"
+                   origin_rpy="0 0 0" origin_xyz="0 0 1"
+                   parent="${l03}"
+                   child="${lee}"
+                   limit_e="10"
+                   limit_l="0"
+                   limit_u="0"
+                   limit_v="0.5"/>
+    <xacro:m_link_cylinder name="${lee}"
+                origin_rpy="0 0 0" origin_xyz="0 0 0"
+                mass = "0.05"
+                ixx="0" ixy="0" ixz="0"
+                iyy="0" iyz="0"
+                izz="0"
+                radius = "0.01"
+                length="0"/>
     <gazebo>
         <plugin name ="gazebo_ros_control" filename="libgazebo_ros_control.so">

File: project_workspace/src/robot_package/urdf/robot_parameters.xacro (robot description, xacro)
@@ -5,3 +5,4 @@
   <xacro:property name="l02" value="link_02" />
   <xacro:property name="l03" value="link_03" />
+  <xacro:property name="lee" value="link_ee" />
 </robot>
